File: MyDoorSensor/MyDoorSensor.brd (EAGLE design)
At the start: 15 x 20 mm, 17 parts, among them IC1 MEGA328P-AU, IC4 ATSHA204A, Q1 BSS84

Commit message: Routed!!
Parts:
- removed JP1: AVR-ISP, pinhead:1X06SMD
- removed JP2: NRF24L01+, pinhead:1X08/1.27
- added U$1: NRF24, mylbr:PINHD-1X08/NRF24
- added U$2: ISP, mylbr:ISP
- moved TP2 56.8 mm to (1.40, 18.6)
- moved R6 44.5 mm to (13.0, 13.7)
- moved Q1 35.7 mm to (13.2, 10.8)
- moved TP1 35.6 mm to (1.40, 1.40)
- moved R3 27.3 mm to (13.9, 6.90), turned to 90 degrees
- moved R1 21.4 mm to (11.9, 6.90), turned to 270 degrees
- moved IC4 11.3 mm to (12.9, 17.9), flipped to the top, turned to 0 degrees
- moved C1 8.66 mm to (1.48, 3.34), flipped to the top, turned to 180 degrees
- moved R2 5.70 mm to (3.70, 17.9), flipped to the top
- moved R4 5.70 mm to (5.73, 17.9), flipped to the top
- moved R5 5.70 mm to (7.77, 17.9), flipped to the top
- moved C7 4.08 mm to (4.93, 1.06)
- moved C2 3.24 mm to (9.51, 17.9), flipped to the top, turned to 90 degrees
- moved IC1 0.70 mm to (5.96, 10.4)
Connections:
- net D10: now also U$1.P$4; no longer JP2.4
- net D2: now also U$1.P$8; no longer JP2.8
- net D9: now also U$1.P$3; no longer JP2.3
- net GND: now also U$1.P$2, U$2.P$6; no longer JP1.6, JP2.2
- net MISO: now also U$1.P$7, U$2.P$1; no longer JP1.1, JP2.7
- net MOSI: now also U$1.P$6, U$2.P$4; no longer JP1.4, JP2.6
- net RST: now also U$2.P$5; no longer JP1.5
- net SCK: now also U$1.P$5, U$2.P$3; no longer JP1.3, JP2.5
- net VCC: now also U$1.P$1, U$2.P$2; no longer JP1.2, JP2.1
Routing:
- net GND: track 0.00 -> 64.4 mm, vias 0 -> 1
- net VCC: track 0.00 -> 62.3 mm, vias 0 -> 5
- net MISO: track 0.00 -> 26.6 mm
- net D10: track 0.00 -> 19.5 mm, vias 0 -> 1
- net D2: track 0.00 -> 18.7 mm, vias 0 -> 1
- net MOSI: track 0.00 -> 18.2 mm, vias 0 -> 1
- net SCK: track 0.00 -> 17.3 mm, vias 0 -> 1
- net D3: track 0.00 -> 15.6 mm
- net A0: track 0.00 -> 11.2 mm, vias 0 -> 2
- net N$4: track 0.00 -> 9.85 mm, vias 0 -> 2
- net RST: track 0.00 -> 9.31 mm, vias 0 -> 1
- net A3: track 0.00 -> 7.19 mm
- net A1: track 0.00 -> 6.20 mm
- net N$2: track 0.00 -> 4.39 mm
- net D9: track 0.00 -> 3.56 mm
