File: MyDoorSensor/MyDoorSensor.sch (EAGLE design)
At the start: 17 parts, among them IC1 MEGA328P-AU, IC4 ATSHA204A, Q1 BSS84

Commit message: Routed!!
Parts:
- removed JP1: AVR-ISP, pinhead:PINHD-1X6SMD
- removed JP2: NRF24L01+, pinhead:PINHD-1X81.27
- added U$1: NRF24, mylbr:NRF24
- added U$2: ISP, mylbr:ISP
Connections:
- net D10: now also U$1.P$4; no longer JP2.4
- net D2: now also U$1.P$8; no longer JP2.8
- net D9: now also U$1.P$3; no longer JP2.3
- net GND: now also U$1.P$2, U$2.P$6; no longer JP1.6, JP2.2
- net MISO: now also U$1.P$7, U$2.P$1; no longer JP1.1, JP2.7
- net MOSI: now also U$1.P$6, U$2.P$4; no longer JP1.4, JP2.6
- net RST: now also U$2.P$5; no longer JP1.5
- net SCK: now also U$1.P$5, U$2.P$3; no longer JP1.3, JP2.5
- net VCC: now also U$1.P$1, U$2.P$2; no longer JP1.2, JP2.1
